File: hardware/pi_avr/RasPiDV.sch (EAGLE design)
At the start: 52 parts, among them Q1 4.9152MHz, Q3 IRLML2060, Q5 2N7002, U1 CML-MICRO_CMX589AE2, U2 MCP6002-I/SN, U3 LD1117-33

Commit message: 
Parts:
- removed C12: 100n, resistor:C-EUC0805
- removed Q1: 4.9152MHz, AIS_Mk2:CRYSTAL_CRYSTALHC49S
- removed U3: LD1117-33, dp_devices:LD1117-3.3SOT223
- added C18, C19: 30p, resistor:C-EUC0805
- added C20, C21: 27n, resistor:C-EUC0805
- added C22: 0.1u, resistor:C-EUC0805
- added D5: Green 0805, adafruit:LEDCHIPLED_0805
- added ISP1: AVRISP-6, adafruit:AVRISP-6
- added J3, J4, J7: JUMPER_SOLDER_1X2, dp_devices:JUMPER_SOLDER_1X2
- added JP5: FTDI connector, adafruit:PINHD-1X6CLEAN
- added JP6: GND, microbuilder:HEADER-1X1ROUND
- added R11, R15: 2K7, adafruit:R-US_M0805
- added R16, R17: 47k, adafruit:R-US_M0805
- added R28: 3K3, adafruit:R-US_M0805
- added R29: 1K5, adafruit:R-US_M0805
- added R7: 1M, adafruit:R-US_M0805
- added U4: ATMEGA328P, SparkFun-DigitalIC:ATMEGA328_SMT
- added U5, U6: (no value), mylibrary:TXS0102DCTR
- added Y1: 4.9152MHz, AIS_Mk2:CRYSTAL_CRYSTALHC49S
- added Y2: 16MHz, AIS_Mk2:CRYSTAL_CRYSTALHC49S
- C14: value 100n -> 0.1u
- R1, R12, R13, R3, R4: value 100k -> 100K; device resistor:R-US_R0805W -> adafruit:R-US_M0805
- R10, R2, R21, R23, R25, R5, R6, R8, R9: device resistor:R-US_R0805W -> adafruit:R-US_M0805
- R14: value 47K -> 47k; device resistor:R-US_R0805W -> adafruit:R-US_M0805
- R22, R26, R27: value 2.7K -> 2K7; device resistor:R-US_R0805W -> adafruit:R-US_M0805
- R24: value 2.2M -> 1M; device resistor:R-US_R0805W -> adafruit:R-US_M0805
- TX: value 200K -> 500K
- U1: device 12_dollar:AIS_MK2_CML-MICRO_CMX589AE2 -> mylibrary:AIS_MK2_CML-MICRO_CMX589AE2
Connections:
- removed net COS_LED: JP1.13, R26.2
- new net DTR: JP1.23, U5.A2
- new net DTR_5: C21.1, JP5.1, U5.B2
- new net MISO: ISP1.MISO, U4.PB4(MISO)
- new net MOSI: ISP1.MOSI, R26.2, U4.PB3(MOSI/OC2)
- new net N$13: C18.2, R7.2, U4.PB6(XTAL1/TOSC1), Y2.2
- new net N$19: J3.2, R28.1, R29.2
- new net N$31: C20.2, U4.AREF
- new net N$32: D5.A, R15.1
- new net N$35: J4.1, R16.1, U6.OE
- new net N$38: J7.1, R17.1, U5.OE
- new net N$8: C19.2, R7.1, U4.PB7(XTAL2/TOSC2), Y2.1
- new net RESET: C21.2, ISP1.RST, R11.2, U4.PC6(/RESET)
- new net RXD: JP1.8, U5.A1
- new net RXD_5: JP5.3, U4.PD0(RXD), U5.B1
- new net SCK: ISP1.SCK, R15.2, U4.PB5(SCK)
- new net SCL: JP1.5, U6.A2
- new net SCL_5: U4.PC5(ADC5/SCL), U6.B2
- new net SDA: JP1.3, U6.A1
- new net SDA_5: U4.PC4(ADC4/SDA), U6.B1
- new net TXD: J3.1, JP1.10
- new net TXD_5: JP5.2, R29.1, U4.PD1(TXD)
- net +3V3: now also J4.2, J7.2, JP1.1, JP1.17, U5.VCCA, U6.VCCA; no longer C14.1, C15.1, C4.1, Q5.D, R10.2, R27.1, R5.2, R6.2, U1.BT, U1.CLKDIVA, U1.CLKDIVB, U1.TXENABLE, U1.VDD, U2P.V+, U3.VOUT
- net +5V: now also C14.1, C15.1, C22.1, C4.1, ISP1.VCC, JP5.4, Q5.D, R10.2, R11.1, R27.1, R5.2, R6.2, U1.BT, U1.CLKDIVA, U1.CLKDIVB, U1.TXENABLE, U1.VDD, U2P.V+, U4.AVCC, U4.VCC@1, U4.VCC@2, U5.VCCB, U6.VCCB; no longer C12.1, U3.VIN
- net COS: now also U4.PD7(AIN1); no longer JP1.11
- net GND: now also C18.1, C19.1, C20.1, C22.2, D5.C, ISP1.GND, JP1.6, JP5.6, JP6.1, R16.2, R17.2, R28.2, U4.AGND, U4.GND@1, U4.GND@2, U5.GND, U6.GND; no longer C12.2, U3.GND
- net N$10: now also Y1.2; no longer Q1.2
- net N$9: now also Y1.1; no longer Q1.1
- net PLLACQ: now also U4.PB1(OC1A); no longer JP1.7
- net PTT: now also U4.PB0(ICP); no longer JP1.15
- net RXCLK: now also U4.PD2(INT0); no longer JP1.22
- net RXDATA: now also U4.PD5(T1); no longer JP1.24
- net RX_SN: now also U4.PD4(XCK/T0); no longer JP1.16
- net TXCLK: now also U4.PD3(INT1); no longer JP1.18
- net TXDATA: now also U4.PD6(AIN0); no longer JP1.26
Other:
- note added: "COS_LED"
- note added: "Status LED"
- moved on the sheet: C1, C10, C11, C13, C14, C15, C16, C17, C2, C3, C4, C5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
