File: hardware/tssop24/tssop24.sch (EAGLE design)
At the start: 3 parts, among them U1 CML-MICRO_CMX589AE2

Commit message: 
Parts:
- U1: device 12_dollar:AIS_MK2_CML-MICRO_CMX589AE2 -> mylibrary:AIS_MK2_CML-MICRO_CMX589AE2
Changed lines of the file:
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@@
 <layer number="54" name="bGND_GNDA" color="7" fill="1" visible="no" active="no"/>
 <layer number="56" name="wert" color="7" fill="1" visible="no" active="no"/>
+<layer number="57" name="tCAD" color="7" fill="1" visible="no" active="no"/>
 <layer number="91" name="Nets" color="2" fill="1" visible="yes" active="yes"/>
 <layer number="92" name="Busses" color="1" fill="1" visible="yes" active="yes"/>
@@
 <layer number="132" name="test" color="7" fill="1" visible="no" active="yes"/>
 <layer number="144" name="Drill_legend" color="7" fill="1" visible="no" active="yes"/>
+<layer number="150" name="Notes" color="7" fill="1" visible="no" active="yes"/>
 <layer number="151" name="HeatSink" color="7" fill="1" visible="yes" active="yes"/>
 <layer number="152" name="_bDocu" color="7" fill="1" visible="no" active="yes"/>
+<layer number="153" name="FabDoc1" color="6" fill="1" visible="no" active="no"/>
+<layer number="154" name="FabDoc2" color="2" fill="1" visible="no" active="no"/>
+<layer number="155" name="FabDoc3" color="7" fill="15" visible="no" active="no"/>
 <layer number="199" name="Contour" color="7" fill="1" visible="no" active="yes"/>
 <layer number="200" name="200bmp" color="7" fill="1" visible="yes" active="yes"/>
@@
 </classes>
 <parts>
-<part name="U1" library="12_dollar" deviceset="AIS_MK2_CML-MICRO_CMX589A" device="E2" value="CML-MICRO_CMX589AE2"/>
+<part name="U1" library="mylibrary" deviceset="AIS_MK2_CML-MICRO_CMX589A" device="E2" value="CML-MICRO_CMX589AE2"/>
 <part name="JP3" library="adafruit" deviceset="PINHD-1X12" device="-CB"/>
 <part name="JP1" library="adafruit" deviceset="PINHD-1X12" device="-CB"/>
