File: hardware/pi/RasPiDV.brd (EAGLE design)
At the start: 33 x 39 mm, 52 parts, among them Q1 4.9152MHz, Q3 IRLML2060, Q5 2N7002, U1 CML-MICRO_CMX589AE2, U2 MCP6002-I/SN, U3 LD1117-33

Commit message: 
Parts:
- moved R14 18.6 mm to (30.5, 17.6)
- moved R10 16.6 mm to (13.9, 18.0), turned to 180 degrees
- moved R21 14.8 mm to (26.3, 18.0), turned to 180 degrees
- moved R6 12.2 mm to (13.9, 19.4)
- moved C4 10.5 mm to (6.88, 13.1), turned to 90 degrees
- moved R5 7.72 mm to (14.0, 20.8), flipped to the bottom, turned to 180 degrees
- moved C1 4.56 mm to (16.4, 7.49)
- moved R3 2.77 mm to (9.91, 21.1)
- moved C6 2.66 mm to (9.88, 20.1)
- moved C5 2.60 mm to (9.50, 13.9), flipped to the bottom, turned to 0 degrees
- moved C8 2.46 mm to (11.9, 7.44)
- moved R4 2.41 mm to (9.86, 18.8)
- moved C13 2.09 mm to (16.9, 23.6)
- moved R24 1.00 mm to (17.0, 21.1)
- moved U1 0.86 mm to (12.7, 13.8)
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Connections:
- net +3V3: now also U1.15
- net GND: no longer U1.15
Routing:
- net GND: track 159.1 -> 0.00 mm, vias 9 -> 8
- net +3V3: track 110.0 -> 74.3 mm, vias 8 -> 5
- net RXDCACQ: track 24.1 -> 3.50 mm
- net VBIAS: track 38.5 -> 24.8 mm
- net N$24: track 18.5 -> 6.23 mm, vias 2 -> 1
- net RXHOLDN: track 19.5 -> 10.4 mm, vias 4 -> 1
- net COS: track 42.8 -> 33.7 mm, vias 0 -> 1
- net COS_LED: track 27.1 -> 22.5 mm, vias 4 -> 2
- net TXCLK: track 15.2 -> 10.5 mm
- net TXOUT: track 56.3 -> 53.1 mm, vias 3 -> 1
- net N$3: track 17.9 -> 14.8 mm, vias 1 -> 0
- net N$9: track 19.1 -> 16.1 mm
- net N$1: track 13.1 -> 10.4 mm
- net RXCLK: track 17.5 -> 14.8 mm, vias 3 -> 1
- net RX_FB: track 17.6 -> 15.1 mm, vias 2 -> 1
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- added copper zone on layer 1, net GND
- added copper zone on layer 16, net GND
- removed copper zone on layer 1, net N$13
- removed copper zone on layer 16, net N$8
Other:
- board text added: "DV"
- board text added: "RasPi"
- board text added: "rev 0.4 (c) 2013"
- board text added: "smd"
- board text removed: "RasPi DV smd"
- board text removed: "rev 0.3 (c) 2013"

Commit message: 
Parts:
- C16: value 100p -> 470p
- D4: value 1N4001 -> DNI
- R23: value 100 -> 330
- R24: value 2.2M -> 1M
- RX: value 200K -> 50K
- TX: value 200K -> 100K
Changed lines of the file:
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@@
 <attribute name="NAME" x="17.8816" y="33.9344" size="0.8128" layer="25" font="vector" ratio="18"/>
 </element>
-<element name="TX" library="pot" package="B25P" value="200K" x="24.2062" y="27.5844" smashed="yes">
+<element name="TX" library="pot" package="B25P" value="100K" x="24.2062" y="27.5844" smashed="yes">
 <attribute name="NAME" x="17.78" y="28.0162" size="1.6764" layer="25" font="vector" ratio="18"/>
 </element>
-<element name="RX" library="pot" package="B25P" value="200K" x="24.2062" y="34.798" smashed="yes">
+<element name="RX" library="pot" package="B25P" value="50K" x="24.2062" y="34.798" smashed="yes">
 <attribute name="NAME" x="17.8562" y="35.2806" size="1.6764" layer="25" font="vector" ratio="18"/>
 </element>
@@
 <attribute name="NAME" x="22.2504" y="22.5806" size="0.8128" layer="25" font="vector" ratio="18"/>
 </element>
-<element name="R23" library="resistor" package="R0805W" value="100" x="21.4122" y="21.082" smashed="yes" rot="MR180">
+<element name="R23" library="resistor" package="R0805W" value="330" x="21.4122" y="21.082" smashed="yes" rot="MR180">
 <attribute name="NAME" x="24.4856" y="21.844" size="0.8128" layer="26" font="vector" ratio="18" rot="MR0"/>
 </element>
-<element name="R24" library="resistor" package="R0805W" value="2.2M" x="17.0434" y="21.082" smashed="yes" rot="R180">
+<element name="R24" library="resistor" package="R0805W" value="1M" x="17.0434" y="21.082" smashed="yes" rot="R180">
 <attribute name="NAME" x="15.0368" y="21.9964" size="0.8128" layer="25" font="vector" ratio="18"/>
 </element>
@@
 <attribute name="NAME" x="30.1498" y="15.4432" size="0.8128" layer="26" font="vector" ratio="18" rot="MR0"/>
 </element>
-<element name="C16" library="resistor" package="C0805" value="100p" x="26.0604" y="20.955" smashed="yes" rot="MR0">
+<element name="C16" library="resistor" package="C0805" value="470p" x="26.0604" y="20.955" smashed="yes" rot="MR0">
 <attribute name="NAME" x="27.813" y="21.971" size="0.8128" layer="26" font="vector" ratio="18" rot="MR0"/>
 </element>
@@
 <attribute name="VALUE" x="5.5626" y="28.9306" size="0.4064" layer="27" ratio="10"/>
 </element>
-<element name="D4" library="diode" package="MICROMELF-R" value="1N4001" x="30.5816" y="21.6916" smashed="yes" rot="MR180">
+<element name="D4" library="diode" package="MICROMELF-R" value="DNI" x="30.5816" y="21.6916" smashed="yes" rot="MR180">
 <attribute name="NAME" x="32.0112" y="22.56" size="0.8128" layer="26" font="vector" ratio="18" rot="MR0"/>
 <attribute name="VALUE" x="29.3806" y="23.7546" size="1.27" layer="28" rot="MR180"/>
